File: RGH3.kicad_sch (KiCad schematic)
At the start: 6 parts

Commit message: Add files via upload
Parts:
- PLL_BYPASS1, POST1, SMC_PLL1, SMC_POST1: footprint TestPoint:TestPoint_Pad_D2.5mm -> TestPoint:TestPoint_Pad_D1.5mm
Changed lines of the file:
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@@
       (effects (font (size 1.27 1.27)) hide)
     )
-    (property "Footprint" "TestPoint:TestPoint_Pad_D2.5mm" (id 2) (at 161.29 118.11 0)
+    (property "Footprint" "TestPoint:TestPoint_Pad_D1.5mm" (id 2) (at 161.29 118.11 0)
       (effects (font (size 1.27 1.27)) hide)
     )
@@
       (effects (font (size 1.27 1.27)) hide)
     )
-    (property "Footprint" "TestPoint:TestPoint_Pad_D2.5mm" (id 2) (at 160.02 90.17 0)
+    (property "Footprint" "TestPoint:TestPoint_Pad_D1.5mm" (id 2) (at 160.02 90.17 0)
       (effects (font (size 1.27 1.27)) hide)
     )
@@
       (effects (font (size 1.27 1.27)) hide)
     )
-    (property "Footprint" "TestPoint:TestPoint_Pad_D2.5mm" (id 2) (at 120.65 118.11 0)
+    (property "Footprint" "TestPoint:TestPoint_Pad_D1.5mm" (id 2) (at 120.65 118.11 0)
       (effects (font (size 1.27 1.27)) hide)
     )
@@
       (effects (font (size 1.27 1.27)) hide)
     )
-    (property "Footprint" "TestPoint:TestPoint_Pad_D2.5mm" (id 2) (at 120.65 90.17 0)
+    (property "Footprint" "TestPoint:TestPoint_Pad_D1.5mm" (id 2) (at 120.65 90.17 0)
       (effects (font (size 1.27 1.27)) hide)
     )
@@
     )
     (path "/1e53d8dc-de34-4621-8a5c-e534a5fcaca7"
-      (reference "PLL_BYPASS1") (unit 1) (value "Conn_01x01") (footprint "TestPoint:TestPoint_Pad_D2.5mm")
+      (reference "PLL_BYPASS1") (unit 1) (value "Conn_01x01") (footprint "TestPoint:TestPoint_Pad_D1.5mm")
     )
     (path "/7cf86a60-529a-49a1-82cb-d1cce9353755"
-      (reference "POST1") (unit 1) (value "Conn_01x01") (footprint "TestPoint:TestPoint_Pad_D2.5mm")
+      (reference "POST1") (unit 1) (value "Conn_01x01") (footprint "TestPoint:TestPoint_Pad_D1.5mm")
     )
     (path "/dd37d2e0-f8a6-4502-90f0-21e1403b1b64"
@@
     )
     (path "/c7fe3c80-68d8-4ee4-bbeb-ab372bec9792"
-      (reference "SMC_PLL1") (unit 1) (value "Conn_01x01") (footprint "TestPoint:TestPoint_Pad_D2.5mm")
+      (reference "SMC_PLL1") (unit 1) (value "Conn_01x01") (footprint "TestPoint:TestPoint_Pad_D1.5mm")
     )
     (path "/e34eff2d-a473-495e-b3e6-3190a6642038"
-      (reference "SMC_POST1") (unit 1) (value "Conn_01x01") (footprint "TestPoint:TestPoint_Pad_D2.5mm")
+      (reference "SMC_POST1") (unit 1) (value "Conn_01x01") (footprint "TestPoint:TestPoint_Pad_D1.5mm")
     )
   )
